Commit message: Cleaned robot URDF

File: src/description/models/core.xacro (robot description, xacro)
@@ -5,7 +5,7 @@
 -->
 <robot xmlns:xacro="http://www.ros.org/wiki/xacro">
-  <xacro:include filename="materials.xacro"/>
-  <xacro:include filename="cylinder.xacro"/>
-  <xacro:include filename="sphere.xacro"/>
+  <xacro:include filename="$(find description)/models/include/materials.xacro"/>
+  <xacro:include filename="$(find description)/models/include/cylinder.xacro"/>
+  <xacro:include filename="$(find description)/models/include/sphere.xacro"/>
   <link name="base_link"/>
   <xacro:CYLINDER

File: src/description/models/gz_sim.xacro (robot description, xacro)
@@ -13,3 +13,68 @@
     </plugin>
   </gazebo>
+  <ros2_control name="manipulator_control" type="system">
+    <hardware>
+        <plugin>gz_ros2_control/GazeboSimSystem</plugin>
+    </hardware>
+    <joint name="joint_01">
+      <command_interface name="position">
+        <param name="min">-3.14</param>
+        <param name="max">3.14</param>
+      </command_interface>
+      <state_interface name="position">
+        <param name="initial_value">0.0</param>
+      </state_interface>
+      <state_interface name="velocity">
+        <param name="initial_value">0.0</param>
+      </state_interface>
+      <state_interface name="effort">
+        <param name="initial_value">0.0</param>
+      </state_interface>
+    </joint>
+    <joint name="joint_23">
+      <command_interface name="position">
+        <param name="min">0.00</param>
+        <param name="max">1.57</param>
+      </command_interface>
+      <state_interface name="position">
+        <param name="initial_value">0.0</param>
+      </state_interface>
+      <state_interface name="velocity">
+        <param name="initial_value">0.0</param>
+      </state_interface>
+      <state_interface name="effort">
+        <param name="initial_value">0.0</param>
+      </state_interface>
+    </joint>
+    <joint name="joint_45">
+      <command_interface name="position">
+        <param name="min">0.00</param>
+        <param name="max">1.57</param>
+      </command_interface>
+      <state_interface name="position">
+        <param name="initial_value">0.0</param>
+      </state_interface>
+      <state_interface name="velocity">
+        <param name="initial_value">0.0</param>
+      </state_interface>
+      <state_interface name="effort">
+        <param name="initial_value">0.0</param>
+      </state_interface>
+    </joint>
+    <joint name="joint_67">
+      <command_interface name="position">
+        <param name="min">0.00</param>
+        <param name="max">1.57</param>
+      </command_interface>
+      <state_interface name="position">
+        <param name="initial_value">0.0</param>
+      </state_interface>
+      <state_interface name="velocity">
+        <param name="initial_value">0.0</param>
+      </state_interface>
+      <state_interface name="effort">
+        <param name="initial_value">0.0</param>
+      </state_interface>
+    </joint>
+  </ros2_control>
 </robot>

File: src/description/models/manipulator.xacro (robot description, xacro)
@@ -7,4 +7,3 @@
   <xacro:include filename="core.xacro"/>
   <xacro:include filename="gz_sim.xacro"/>
-  <xacro:include filename="ros2_control.xacro"/>
 </robot>
